File: bikeleds/bikeleds.kicad_pcb (KiCad board)
At the start: 2 copper layers, 19.5 x 26.8 mm, 20 parts, among them J1 USB_B_Micro, J2 Conn_01x03_Pin, U1 ATSAMD51G19A-MU, U2 AP2112K-3.3, U3 74AHCT1G125, U4 TSOP77438TT

Commit message: v2 of bikeleds
Parts:
- removed TP1, TP2, TP3, TP4, TP5: TestPoint, TestPoint:TestPoint_Pad_D1.5mm
- added J3: Conn_01x06, Connector_PinSocket_2.54mm:PinSocket_1x06_P2.54mm_Vertical, F.Cu at (140.6, 89.9)
- C8: footprint Capacitor_SMD:C_0805_2012Metric -> Capacitor_SMD:C_0603_1608Metric
- moved U3 18.3 mm to (156.2, 102.0), turned to 90 degrees
- moved C2 1.86 mm to (153.0, 102.1)
- moved C8 1.25 mm to (143.4, 94.3), turned to -90 degrees
- moved C1 1.14 mm to (143.7, 102.1)
- moved C7 1.05 mm to (155.3, 95.4)
Connections:
- J2 pad 1: VBUS -> GND
- J2 pad 3: GND -> VBUS
Routing:
- net VBUS: track 35.3 -> 49.5 mm
- net /RESET: track 5.40 -> 19.2 mm
- net /LEDS_OUT: track 9.90 -> 22.5 mm, vias 0 -> 1
- net /SWCLK: track 8.55 -> 15.8 mm
- net +3V3: track 51.7 -> 47.0 mm
- net /LEDS_IN: track 9.32 -> 14.0 mm
- net GND: track 34.8 -> 38.2 mm, vias 13 -> 12
- net /SWDIO: track 13.1 -> 15.6 mm
Other:
- board text added: "3v3"
- board text added: "CLK"
- board text added: "DIO"
- board text added: "GND"
- board text added: "RST"
- board text added: "v2"
- board text removed: "+"
- board text removed: "C"
- board text removed: "D"
- board text removed: "G"
- board text removed: "R"
