File: bikeleds/bikeleds.kicad_sch (KiCad schematic)
At the start: 20 parts, among them J2 Conn_01x03_Pin, J3 USB_B_Micro, U1 ATSAMD51G19A-MU, U2 AP2112K-3.3, U3 74AHCT1G125, U4 TSOP77438TT

Commit message: v2 of bikeleds
Parts:
- removed TP1, TP2, TP3, TP4, TP5: TestPoint, TestPoint:TestPoint_Pad_D1.5mm, symbol Connector:TestPoint
- added J3: Conn_01x06, Connector_PinSocket_2.54mm:PinSocket_1x06_P2.54mm_Vertical, symbol Connector_Generic:Conn_01x06
- C8: footprint Capacitor_SMD:C_0805_2012Metric -> Capacitor_SMD:C_0603_1608Metric
Connections:
- net +3V3: now also J3.4 (Pin_4)
- net GND: now also J2.1 (Pin_1), J3.5 (Pin_5); no longer J2.3 (Pin_3)
- net RESET: now also J3.3 (Pin_3)
- net SWCLK: now also J3.2 (Pin_2)
- net SWDIO: now also J3.1 (Pin_1)
- net VBUS: now also J2.3 (Pin_3); no longer J2.1 (Pin_1)
- no-connect marks 34 -> 35
