File: heads-v3/heads-v3.kicad_pcb (KiCad board)
At the start: 2 copper layers, 23 x 17.5 mm, 8 parts, among them J1 GPIO, J2 Conn_01x02_Pin

Commit message: v4
Parts:
- removed MH1: MountingHole_2.7mm_M2.5, MountingHole:MountingHole_2.7mm_M2.5
- added C3: 0.1uF, Capacitor_SMD:C_0805_2012Metric, F.Cu at (113.5, 82.1)
- added C4: 10uF, Capacitor_SMD:C_1206_3216Metric, F.Cu at (120.8, 82.8)
- added C5: 10uF, Capacitor_SMD:C_1206_3216Metric, F.Cu at (118.2, 82.8)
- added C6: 10uF, Capacitor_SMD:C_1206_3216Metric, F.Cu at (115.8, 82.8)
- added C7: 0.1uF, Capacitor_SMD:C_0805_2012Metric, F.Cu at (104.5, 76.2)
- added C8: 10uF, Capacitor_SMD:C_1206_3216Metric, F.Cu at (104.0, 74.0)
- added C9: 10uF, Capacitor_SMD:C_1206_3216Metric, F.Cu at (111.5, 54.5)
- added H1: MountingHole, MountingHole:MountingHole_2.7mm_M2.5, F.Cu at (103.5, 47.5)
- added H2: MountingHole, MountingHole:MountingHole_2.7mm_M2.5, F.Cu at (103.5, 96.5)
- added J3: Conn_01x03_Pin, Connector_PinHeader_2.54mm:PinHeader_1x03_P2.54mm_Vertical_SMD_Pin1Left, F.Cu at (118.0, 54.9)
- added J4: Conn_01x04_Pin, Connector_PinHeader_2.54mm:PinHeader_1x04_P2.54mm_Vertical_SMD_Pin1Left, F.Cu at (116.8, 64.3)
- added J5: Conn_01x02, TerminalBlock_4Ucon:TerminalBlock_4Ucon_1x02_P3.50mm_Horizontal, F.Cu at (104.2, 64.0)
- added J6: Conn_01x04, Connector_JST:JST_SH_BM04B-SRSS-TB_1x04-1MP_P1.00mm_Vertical, F.Cu at (102.7, 54.5)
- added R2: 0.2, Resistor_SMD:R_0805_2012Metric, F.Cu at (121.2, 72.9)
- added R3: 0.2, Resistor_SMD:R_0805_2012Metric, F.Cu at (121.2, 76.4)
- added R4: 100k, Resistor_SMD:R_0805_2012Metric, F.Cu at (106.6, 86.3)
- added R5: 1k, Resistor_SMD:R_0805_2012Metric, F.Cu at (113.3, 95.0)
- added U1: ATSAMD09D14A-M, Package_DFN_QFN:QFN-24-1EP_4x4mm_P0.5mm_EP2.6x2.6mm, F.Cu at (110.2, 75.1)
- added U3: DRV8833PW, Package_SO:TSSOP-16_4.4x5mm_P0.65mm, F.Cu at (117.3, 74.8)
- added U4: 74AHCT1G125, Package_TO_SOT_SMD:SOT-353_SC-70-5, F.Cu at (108.2, 54.0)
- J2: value Conn_01x02_Pin -> Conn_01x02; footprint TerminalBlock_4Ucon:TerminalBlock_4Ucon_1x02_P3.50mm_Horizontal -> Connector_PinHeader_2.54mm:PinHeader_1x06_P2.54mm_Vertical
- R1: value R -> 0.15
- moved J2 43.4 mm to (107.8, 98.2), turned to 90 degrees
- moved C1 37.4 mm to (103.0, 90.5), turned to 90 degrees
- moved U2 31.4 mm to (102.4, 86.2), turned to 90 degrees
- moved L1 30.5 mm to (104.8, 81.0), turned to 90 degrees
- moved C2 27.1 mm to (108.4, 81.2)
- moved R1 25.7 mm to (101.2, 81.7), turned to 90 degrees
Connections:
- J1 pad 10: unconnected-(J1-Pin_10-Pad10) -> (no net)
- J1 pad 11: unconnected-(J1-Pin_11-Pad11) -> (no net)
- J1 pad 12: /PWM -> (no net)
- J1 pad 3: unconnected-(J1-Pin_3-Pad3) -> /SDA
- J1 pad 5: unconnected-(J1-Pin_5-Pad5) -> /SCL
- J1 pad 7: unconnected-(J1-Pin_7-Pad7) -> /SEESAW_RST
- J1 pad 9: GND -> (no net)
- J2 pad 1: /+LED -> +3V3
- J2 pad 2: /-LED -> GND
- U2 pad 2: +3V3 -> /IR_EN
Routing:
- net +3V3: track 15.4 -> 123.0 mm, vias 2 -> 4
- net /SEESAW_RST: track 0.00 -> 62.6 mm, vias 0 -> 6
- net +5V: track 32.9 -> 83.9 mm, vias 0 -> 2
- net /SCL: track 0.00 -> 41.3 mm, vias 0 -> 5
- net /SDA: track 0.00 -> 36.1 mm, vias 0 -> 4
- net /SWCLK: track 0.00 -> 30.2 mm, vias 0 -> 4
- net /SWDIO: track 0.00 -> 29.5 mm, vias 0 -> 4
- net GND: track 5.27 -> 29.5 mm, vias 0 -> 13
- net /IR_EN: track 0.00 -> 23.9 mm, vias 0 -> 4
- net /LEDS: track 0.00 -> 23.2 mm, vias 0 -> 2
- net Net-(J3-Pin_2): track 0.00 -> 18.4 mm
- net /-LED: track 12.8 -> 23.6 mm
- net /AOUT1: track 0.00 -> 9.71 mm
- net /BOUT2: track 0.00 -> 9.68 mm
- net /AIN1: track 0.00 -> 9.58 mm
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Other:
- board size 23 x 17.5 mm -> 22.3 x 56 mm
- board text added: "+"
- board text added: "-"
- board text added: "3v3"
- board text added: "CLK"
- board text added: "DIO"
- board text added: "GND"
- board text added: "RST"
- board text added: "The Heads v04"
- board text removed: "DISPLAY (OPTIONAL)"
- board text removed: "LED Driver v0.1"
