File: heads-v3/heads-v3.kicad_sch (KiCad schematic)
At the start: 7 parts, among them J1 GPIO, J2 Conn_01x02_Pin

Commit message: v4
Parts:
- removed J2: Conn_01x02_Pin, TerminalBlock_4Ucon:TerminalBlock_4Ucon_1x02_P3.50mm_Horizontal, symbol Connector:Conn_01x02_Socket
- added C3, C7: 0.1uF, Capacitor_SMD:C_0805_2012Metric, symbol Device:C
- added C4, C5, C6, C8, C9: 10uF, Capacitor_SMD:C_1206_3216Metric, symbol Device:C
- added H1, H2: MountingHole, MountingHole:MountingHole_2.7mm_M2.5, symbol Mechanical:MountingHole
- added J2: Conn_01x02, Connector_PinHeader_2.54mm:PinHeader_1x06_P2.54mm_Vertical, symbol Connector_Generic:Conn_01x06
- added J3: Conn_01x03_Pin, Connector_PinHeader_2.54mm:PinHeader_1x03_P2.54mm_Vertical_SMD_Pin1Left, symbol Connector:Conn_01x03_Pin
- added J4: Conn_01x04_Pin, Connector_PinHeader_2.54mm:PinHeader_1x04_P2.54mm_Vertical_SMD_Pin1Left, symbol Connector:Conn_01x04_Pin
- added J5: Conn_01x02, TerminalBlock_4Ucon:TerminalBlock_4Ucon_1x02_P3.50mm_Horizontal, symbol Connector_Generic:Conn_01x02
- added J6: Conn_01x04, Connector_JST:JST_SH_BM04B-SRSS-TB_1x04-1MP_P1.00mm_Vertical, symbol Connector_Generic:Conn_01x04
- added R2, R3: 0.2, Resistor_SMD:R_0805_2012Metric, symbol Device:R
- added R4: 100k, Resistor_SMD:R_0805_2012Metric, symbol Device:R
- added R5: 1k, Resistor_SMD:R_0805_2012Metric, symbol Device:R
- added U1: ATSAMD09D14A-M, Package_DFN_QFN:QFN-24-1EP_4x4mm_P0.5mm_EP2.6x2.6mm, symbol MCU_Microchip_SAMD:ATSAMD09D14A-M
- added U3: DRV8833PW, Package_SO:TSSOP-16_4.4x5mm_P0.65mm, symbol Driver_Motor:DRV8833PW
- added U4: 74AHCT1G125, Package_TO_SOT_SMD:SOT-353_SC-70-5, symbol 74xGxx:74AHCT1G125
- R1: value R -> 0.15
Connections:
- net +3V3: now also C7.1, C8.1, J2.1 (Pin_1), J6.2 (Pin_2), R5.2, U1.24 (VDD), U3.1 (nSLEEP); no longer U2.2 (EN)
- net +5V: now also C3.1, C5.1, C6.1, C9.1, J3.1 (Pin_1), U3.12 (VM), U4.5 (VCC)
- net +LED: now also J5.2 (Pin_2)
- net -LED: now also J5.1 (Pin_1)
- net GND: now also C4.2, C5.2, C6.2, C7.2, C8.2, C9.2, J2.2 (Pin_2), J3.3 (Pin_3), J6.1 (Pin_1), R2.1, R3.1, R4.1, U1.23 (GND), U1.25 (GND), U3.13 (GND), U4.1, U4.3 (GND); no longer J1.9 (Pin_9)
- net PWM: now also U1.5 (PA06); no longer J1.12 (Pin_12)
- net SDA: now reaches J1.3 (Pin_3)
- net SDA: now also J6.3 (Pin_3), U1.15 (PA22)
- net SCL: now reaches J1.5 (Pin_5)
- net SCL: now also J6.4 (Pin_4), U1.16 (PA23)
- net SEESAW_RST: now reaches J1.7 (Pin_7)
- net SEESAW_RST: now also J2.5 (Pin_5), U1.18 (PA28/~{RST})
- new net: J3.2 (Pin_2), U4.4
- new net AIN1: U1.11 (PA14), U3.16 (AIN1)
- new net AIN2: U1.10 (PA11), U3.15 (AIN2)
- new net AISEN: R2.2, U3.3 (AISEN)
- new net AOUT1: J4.4 (Pin_4), U3.2 (AOUT1)
- new net AOUT2: J4.3 (Pin_3), U3.4 (AOUT2)
- new net BIN1: U1.8 (PA09/XOUT), U3.9 (BIN1)
- new net BIN2: U1.9 (PA10), U3.10 (BIN2)
- new net BISEN: R3.2, U3.6 (BISEN)
- new net BOUT1: J4.1 (Pin_1), U3.7 (BOUT1)
- new net BOUT2: J4.2 (Pin_2), U3.5 (BOUT2)
- new net IR_EN: R4.2, U1.12 (PA15), U2.2 (EN)
- new net LEDS: U1.22 (PA25), U4.2
- new net SWCLK: J2.4 (Pin_4), R5.1, U1.19 (PA30/SWCLK)
- new net SWDIO: J2.3 (Pin_3), U1.20 (PA31/SWDIO)
- new net VCP: C3.2, U3.11 (VCP)
- new net VINT: C4.1, U3.14 (VINT)
- no-connect marks 6 -> 12
Other:
- moved on the sheet: C1
