File: nes-controller-v3/nes-controller-v3.kicad_pcb (KiCad board)
At the start: 2 copper layers, 58.2 x 20.1 mm, 16 parts, among them J1 USB_B_Micro, J3 Conn_01x06, U2 AP2112K-3.3, U7 ATSAMD21E18A-A

Commit message: ship
Parts:
- removed R1, R2: 10k, Resistor_SMD:R_0805_2012Metric
- added D1: D, Diode_SMD:D_0805_2012Metric, F.Cu at (149.2, 72.6)
- added D2: D, Diode_SMD:D_0805_2012Metric, F.Cu at (130.3, 71.3)
- added J2: NES, Connector_Wire:SolderWire-0.15sqmm_1x05_P4mm_D0.5mm_OD1.5mm_Relief, B.Cu at (145.5, 71.2)
- added U1: SN74LVC125ADR, Minor_Industries:SN74LVC125ADR, F.Cu at (157.4, 71.5)
- J1: moved to F.Cu
- moved J1 33.7 mm to (109.0, 74.8), turned to -90 degrees
- moved C7 28.9 mm to (132.8, 75.7), turned to 90 degrees
- moved C2 24.7 mm to (136.2, 75.6), turned to 90 degrees
- moved U2 15.8 mm to (140.6, 75.0), turned to 180 degrees
- moved C4 13.2 mm to (126.5, 75.8), turned to 0 degrees
- moved C8 13.0 mm to (127.2, 65.8), turned to -90 degrees
- moved C1 6.15 mm to (145.6, 75.4), turned to -90 degrees
- moved U4 5.83 mm to (121.1, 74.7)
- moved U7 5.60 mm to (120.8, 69.5), turned to 180 degrees
- moved H1 5.22 mm to (110.3, 81.8)
- moved H3 4.73 mm to (140.4, 66.8)
- moved U3 3.33 mm to (159.7, 74.7)
- moved H2 2.61 mm to (170.9, 81.8)
- moved J3 2.02 mm to (166.1, 65.7)
Connections:
- net /C renamed /PAD_CLOCK
- net /D1 renamed /PAD_DATA_1
- net /D2 renamed /PAD_DATA_2
- net /L renamed /PAD_LATCH
- C1 pad 1: VBUS -> /+5V*
- U2 pad 1: VBUS -> /+5V*
- U2 pad 3: VBUS -> /+5V*
- U7 pad 12: unconnected-(U7-PA09-Pad12) -> /NES_DATA
- U7 pad 13: unconnected-(U7-PA10-Pad13) -> /NES_LATCH_3V
- U7 pad 14: unconnected-(U7-PA11-Pad14) -> /NES_CLOCK_3V
Routing:
- net /NES_CLOCK_3V: track 0.00 -> 57.2 mm, vias 0 -> 4
- net /NES_LATCH_3V: track 0.00 -> 52.4 mm, vias 0 -> 2
- net /NES_CLOCK_5V: track 0.00 -> 26.3 mm
- net /NES_DATA: track 0.00 -> 25.9 mm, vias 0 -> 2
- net /+5V*: track 0.00 -> 22.9 mm
- net /NES_LATCH_5V: track 0.00 -> 20.7 mm
- net /RESET: track 36.6 -> 57.2 mm, vias 3 -> 4
- net /SWDIO: track 46.9 -> 64.2 mm, vias 3 -> 0
- net /SWCLK: track 41.4 -> 57.6 mm, vias 2 -> 4
- net GND: track 12.9 -> 26.7 mm, vias 7 -> 10
- net /D+: track 19.4 -> 5.76 mm, vias 1 -> 0
- net +3V3: track 79.0 -> 92.0 mm, vias 0 -> 6
- net /D-: track 18.6 -> 5.82 mm, vias 1 -> 0
- net /PAD_CLOCK: track 49.8 -> 55.5 mm, vias 1 -> 3
- net /PAD_LATCH: track 49.3 -> 53.9 mm, vias 1 -> 2
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Other:
- board size 58.2 x 20.1 mm -> 66.1 x 20.1 mm
- board text added: "NES Controllers v0.2"
- board text removed: "3V3"
- board text removed: "GND"
- board text removed: "NES Controllers v0.1"
