File: nes-controller-v3/nes-controller-v3.kicad_pcb (KiCad board)
At the start: 2 copper layers, 66.1 x 20.1 mm, 18 parts, among them J1 USB_B_Micro, J2 NES, J3 Conn_01x06, U1 SN74LVC125ADR, U2 AP2112K-3.3, U7 ATSAMD21E18A-A

Commit message: fix pour issue
Routing:
- removed copper zone on F.Cu, net GND
Other:
- board text added: "NES Controllers v0.3"
- board text removed: "NES Controllers v0.2"
Changed lines of the file:
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@@
     (effects (font (size 0.8 0.8) (thickness 0.15)) (justify left bottom))
   )
-  (gr_text "NES Controllers v0.2" (at 133.01 84.025) (layer "F.SilkS")
+  (gr_text "NES Controllers v0.3" (at 133.01 84.025) (layer "F.SilkS")
     (effects (font (size 1 1) (thickness 0.2) bold italic) (justify left bottom))
   )
@@
   (segment (start 117.21 73.225) (end 118.01 72.425) (width 0.3) (layer "B.Cu") (net 43))
   (segment (start 116.81 73.225) (end 117.21 73.225) (width 0.3) (layer "B.Cu") (net 43))
-  (zone (net 27) (net_name "GND") (layer "F.Cu") (hatch edge 0.5)
-    (connect_pads (clearance 0.5))
-    (min_thickness 0.25) (filled_areas_thickness no)
-    (fill yes (thermal_gap 0.5) (thermal_bridge_width 0.5))
-    (polygon
-      (pts
-        (xy 104.3 59.7)
-        (xy 180.6 59.9)
-        (xy 180.8 103.1)
-        (xy 103.2 103.4)
-      )
-    )
-  )
   (zone (net 27) (net_name "GND") (layer "B.Cu") (hatch edge 0.5)
     (priority 1)
