File: nes-controller-v3/nes-controller-v3.kicad_sch (KiCad schematic)
At the start: 16 parts, among them J3 Conn_01x06, J3 USB_B_Micro, U1 ATSAMD21E18A-A, U2 AP2112K-3.3

Commit message: ship
Parts:
- removed R1, R2: 10k, Resistor_SMD:R_0805_2012Metric, symbol Device:R
- added D1, D2: D, Diode_SMD:D_0805_2012Metric, symbol Device:D
- added J2: NES, Connector_Wire:SolderWire-0.15sqmm_1x05_P4mm_D0.5mm_OD1.5mm_Relief, symbol Connector:Conn_01x05_Pin
- added U1: SN74LVC125ADR, Minor_Industries:SN74LVC125ADR, symbol Minor_Industries:SN74LVC125ADR
Connections:
- net +3V3: now also U1.10 (*3OE), U1.13 (*4OE), U1.14 (VCC)
- net GND: now also J2.2 (Pin_2), U1.1 (*1OE), U1.4 (*2OE), U1.7 (GND)
- net VBUS: now also D2.2 (A); no longer C1.1, U2.1 (VIN), U2.3 (EN)
- net NES_DATA: now reaches U1.12 (PA09)
- net NES_DATA: now also J2.3 (Pin_3)
- net NES_LATCH_3V: now reaches U1.13 (PA10)
- net NES_LATCH_3V: now also U1.3 (1Y)
- net NES_CLOCK_3V: now reaches U1.14 (PA11)
- net NES_CLOCK_3V: now also U1.6 (2Y)
- net C renamed PAD_CLOCK
- net D1 renamed PAD_DATA_1
- net D2 renamed PAD_DATA_2
- net L renamed PAD_LATCH
- new net +5V*: C1.1, D1.1 (K), D2.1 (K), U2.1 (VIN), U2.3 (EN)
- new net NES_5V: D1.2 (A), J2.1 (Pin_1)
- new net NES_CLOCK_5V: J2.5 (Pin_5), U1.5 (2A)
- new net NES_LATCH_5V: J2.4 (Pin_4), U1.2 (1A)
- no-connect marks 21 -> 22
Other:
- note added: "TODO: breakout/test pins TODO: check diode package sizes"
