File: nes-controller-v4/nes-controller-v4.kicad_sch (KiCad schematic)
At the start: 18 parts, among them J2 NES, J3 Conn_01x06, J3 USB_B_Micro, U1 ATSAMD21E18A-A, U1 SN74LVC125ADR, U2 AP2112K-3.3

Commit message: v4
Parts:
- removed D1, D2: D, Diode_SMD:D_0805_2012Metric, symbol Device:D
- added R2, R3, R4: 10k, Resistor_SMD:R_0805_2012Metric, symbol Device:R
Connections:
- net NES_5V is gone; now on net +5V: J2.1 (Pin_1)
- net VBUS is gone; now on net +5V: J3.1 (VBUS)
- net +3V3: now also R2.1, R3.1, R4.1
- net NES_DATA: now also R4.2
- net PAD_DATA_1: now also R2.2
- net PAD_DATA_2: now also R3.2
- net +5V* renamed +5V
Other:
- moved on the sheet: J2
