File: nes-controller-v4/nes-controller-v4.kicad_pcb (KiCad board)
At the start: 2 copper layers, 66.1 x 20.1 mm, 18 parts, among them J1 USB_B_Micro, J2 NES, J3 Conn_01x06, U1 SN74LVC125ADR, U2 AP2112K-3.3, U7 ATSAMD21E18A-A

Commit message: v4
Parts:
- removed D1, D2: D, Diode_SMD:D_0805_2012Metric
- added R2: 10k, Resistor_SMD:R_0805_2012Metric, F.Cu at (165.7, 76.5)
- added R3: 10k, Resistor_SMD:R_0805_2012Metric, F.Cu at (119.0, 83.5)
- added R4: 10k, Resistor_SMD:R_0805_2012Metric, F.Cu at (136.1, 67.9)
Connections:
- C1 pad 1: /+5V* -> +5V
- J1 pad 1: VBUS -> +5V
- J2 pad 1: /NES_5V -> +5V
- U2 pad 1: /+5V* -> +5V
- U2 pad 3: /+5V* -> +5V
Routing:
- net +5V: track 0.00 -> 44.5 mm, vias 0 -> 3
- net VBUS: track 25.0 -> 0.00 mm, vias 2 -> 0
- net /+5V*: track 22.9 -> 0.00 mm
- net /PAD_DATA_1: track 38.6 -> 55.8 mm, vias 0 -> 1
- net +3V3: track 92.0 -> 106.6 mm, vias 6 -> 7
- net /NES_DATA: track 25.9 -> 31.2 mm, vias 2 -> 3
- net /PAD_DATA_2: track 18.7 -> 22.8 mm
- net /NES_5V: track 3.93 -> 0.00 mm
Other:
- board text added: "NES Controllers v0.4"
- board text removed: "NES Controllers v0.3"

Commit message: fix
Parts:
- moved R4 2.10 mm to (136.2, 65.8)
Routing:
- net /NES_DATA: track 31.2 -> 32.3 mm
- net +3V3: track 106.6 -> 107.3 mm
Changed lines of the file:
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@@
   )
   (footprint "Resistor_SMD:R_0805_2012Metric" (layer "F.Cu")
-    (at 136.11 67.875 -90)
+    (at 136.16 65.775 -90)
     (descr "Resistor SMD 0805 (2012 Metric), square (rectangular) end terminal, IPC_7351 nominal, (Body size source: IPC-SM-782 page 72, https://www.pcb-3d.com/wordpress/wp-content/uploads/ipc-sm-782a_amendment_1_and_2.pdf), generated with kicad-footprint-generator")
     (tags "resistor")
@@
   (segment (start 139.19 70.025) (end 140.39 71.225) (width 0.3) (layer "F.Cu") (net 7))
   (segment (start 136.65 70.727943) (end 137.352943 70.025) (width 0.3) (layer "F.Cu") (net 7))
-  (segment (start 137.86 68.7755) (end 136.122 68.7755) (width 0.25) (layer "F.Cu") (net 7))
   (segment (start 128.31 68.425) (end 130.16 70.275) (width 0.3) (layer "F.Cu") (net 7))
   (segment (start 132.0475 70.622811) (end 132.0475 71.313972) (width 0.3) (layer "F.Cu") (net 7))
-  (segment (start 136.122 68.7755) (end 136.11 68.7875) (width 0.25) (layer "F.Cu") (net 7))
   (segment (start 121.0595 66.3505) (end 121.16 66.25) (width 0.3) (layer "F.Cu") (net 7))
   (segment (start 121.16 66.25) (end 121.16 65.275) (width 0.3) (layer "F.Cu") (net 7))
@@
   (segment (start 136.65 71.685) (end 136.65 70.727943) (width 0.3) (layer "F.Cu") (net 7))
   (segment (start 133.158528 72.425) (end 135.696523 72.425) (width 0.3) (layer "F.Cu") (net 7))
+  (segment (start 137.86 68.7755) (end 136.16 67.0755) (width 0.25) (layer "F.Cu") (net 7))
   (segment (start 121.0595 66.925) (end 121.0595 66.3505) (width 0.3) (layer "F.Cu") (net 7))
   (segment (start 132.0475 71.313972) (end 133.158528 72.425) (width 0.3) (layer "F.Cu") (net 7))
@@
   (segment (start 135.935 72.4) (end 136.65 71.685) (width 0.3) (layer "F.Cu") (net 7))
   (segment (start 135.721523 72.4) (end 135.935 72.4) (width 0.3) (layer "F.Cu") (net 7))
+  (segment (start 136.16 67.0755) (end 136.16 66.6875) (width 0.25) (layer "F.Cu") (net 7))
   (segment (start 137.352943 70.025) (end 139.19 70.025) (width 0.3) (layer "F.Cu") (net 7))
   (segment (start 131.699689 70.275) (end 132.0475 70.622811) (width 0.3) (layer "F.Cu") (net 7))
@@
   (segment (start 164.1595 75.575) (end 165.685 75.575) (width 0.3) (layer "F.Cu") (net 28))
   (segment (start 120.762743 79.75) (end 123.087743 77.425) (width 0.25) (layer "F.Cu") (net 28))
+  (segment (start 135.288512 64.8625) (end 133.71 66.441012) (width 0.25) (layer "F.Cu") (net 28))
   (segment (start 127.21 64.875) (end 132.143988 64.875) (width 0.5) (layer "F.Cu") (net 28))
   (segment (start 133.722762 75.694004) (end 133.722762 75.762238) (width 0.5) (layer "F.Cu") (net 28))
@@
   (segment (start 155.8688 70.725) (end 154.88 69.7362) (width 0.3) (layer "F.Cu") (net 28))
   (segment (start 140.2225 76.725) (end 139.4725 75.975) (width 0.5) (layer "F.Cu") (net 28))
-  (segment (start 135.9475 67.125) (end 133.71 67.125) (width 0.25) (layer "F.Cu") (net 28))
   (segment (start 165.685 75.575) (end 165.71 75.55) (width 0.3) (layer "F.Cu") (net 28))
   (segment (start 153.61 69.025) (end 154.88 69.025) (width 0.3) (layer "F.Cu") (net 28))
@@
   (segment (start 158.7024 70.725) (end 160.6006 72.6232) (width 0.3) (layer "F.Cu") (net 28))
   (segment (start 149.649026 75.025) (end 144.595051 75.025) (width 0.5) (layer "F.Cu") (net 28))
-  (segment (start 136.11 66.9625) (end 135.9475 67.125) (width 0.25) (layer "F.Cu") (net 28))
   (segment (start 158.49 70.725) (end 158.69 70.525) (width 0.3) (layer "F.Cu") (net 28))
   (segment (start 151.585421 73.088605) (end 149.649026 75.025) (width 0.5) (layer "F.Cu") (net 28))
@@
   (segment (start 121.96 69.994576) (end 122.11 69.844576) (width 0.5) (layer "F.Cu") (net 28))
   (segment (start 122.11 68.456371) (end 123.56 67.006371) (width 0.5) (layer "F.Cu") (net 28))
+  (segment (start 136.16 64.8625) (end 135.288512 64.8625) (width 0.25) (layer "F.Cu") (net 28))
   (segment (start 133.71 66.441012) (end 133.71 67.125) (width 0.5) (layer "F.Cu") (net 28))
   (segment (start 133.71 67.125) (end 133.71 71.7255) (width 0.5) (layer "F.Cu") (net 28))
